Commit message: Initial commit

File: legged_gym/resources/robots/N1/N1_rotor.urdf (robot description, URDF)
Before this commit: robot N1, 29 links, 28 joints
Links:
- link left_end_effector_link: geometry visual mesh filename=meshes/left_end_effector_link.STL
- link left_hand_yaw_link: geometry visual mesh filename=meshes/left_hand_yaw_link.STL
- link left_thigh_roll_link: geometry visual mesh filename=meshes/left_thigh_roll_link.STL
- link left_thigh_yaw_link: geometry visual mesh filename=meshes/left_thigh_yaw_link.STL
- link left_upper_arm_roll_link: geometry visual mesh filename=meshes/left_upper_arm_roll_link.STL
- link left_upper_arm_yaw_link: geometry visual mesh filename=meshes/left_upper_arm_yaw_link.STL
- link right_end_effector_link: geometry visual mesh filename=meshes/right_end_effector_link.STL
- link right_hand_yaw_link: geometry visual mesh filename=meshes/right_hand_yaw_link.STL
- link right_thigh_roll_link: geometry visual mesh filename=meshes/right_thigh_roll_link.STL
- link right_thigh_yaw_link: geometry visual mesh filename=meshes/right_thigh_yaw_link.STL
- link right_upper_arm_roll_link: geometry visual mesh filename=meshes/right_upper_arm_roll_link.STL
- link right_upper_arm_yaw_link: geometry visual mesh filename=meshes/right_upper_arm_yaw_link.STL
- link torso_link: geometry collision cylinder length=0.15 radius=0.08; collision sphere radius=0.08
- link waist_yaw_link: geometry visual mesh filename=meshes/waist_yaw_link.STL

File: legged_gym/resources/robots/g1/g1_12dof_with_hand.urdf (robot description, URDF)
Before this commit: robot g1_29dof_with_hand_rev_1_0, 53 links, 52 joints
Links:
- link head_link: geometry visual mesh filename=meshes/head_link.STL
- link left_ankle_pitch_link: geometry visual mesh filename=meshes/left_ankle_pitch_link.STL
- link left_elbow_link: geometry visual mesh filename=meshes/left_elbow_link.STL
- link left_hand_index_0_link: geometry visual mesh filename=meshes/left_hand_index_0_link.STL
- link left_hand_index_1_link: geometry visual mesh filename=meshes/left_hand_index_1_link.STL
- link left_hand_middle_0_link: geometry visual mesh filename=meshes/left_hand_middle_0_link.STL
- link left_hand_middle_1_link: geometry visual mesh filename=meshes/left_hand_middle_1_link.STL
- link left_hand_palm_link: geometry visual mesh filename=meshes/left_hand_palm_link.STL
- link left_hand_thumb_0_link: geometry visual mesh filename=meshes/left_hand_thumb_0_link.STL
- link left_hand_thumb_1_link: geometry visual mesh filename=meshes/left_hand_thumb_1_link.STL
- link left_hand_thumb_2_link: geometry visual mesh filename=meshes/left_hand_thumb_2_link.STL
- link left_hip_pitch_link: geometry visual mesh filename=meshes/left_hip_pitch_link.STL
- link left_hip_roll_link: geometry visual mesh filename=meshes/left_hip_roll_link.STL
- link left_hip_yaw_link: geometry visual mesh filename=meshes/left_hip_yaw_link.STL
- link left_knee_link: geometry collision cylinder length=0.2 radius=0.05; visual mesh filename=meshes/left_knee_link.STL
- link left_shoulder_pitch_link: geometry visual mesh filename=meshes/left_shoulder_pitch_link.STL
- link left_shoulder_roll_link: geometry visual mesh filename=meshes/left_shoulder_roll_link.STL
- link left_shoulder_yaw_link: geometry visual mesh filename=meshes/left_shoulder_yaw_link.STL
- link left_wrist_pitch_link: geometry visual mesh filename=meshes/left_wrist_pitch_link.STL
- link left_wrist_roll_link: geometry visual mesh filename=meshes/left_wrist_roll_link.STL
- link left_wrist_yaw_link: geometry visual mesh filename=meshes/left_wrist_yaw_link.STL
- link logo_link: geometry visual mesh filename=meshes/logo_link.STL
- link pelvis_contour_link: geometry visual mesh filename=meshes/pelvis_contour_link.STL
- link right_ankle_pitch_link: geometry visual mesh filename=meshes/right_ankle_pitch_link.STL
- link right_elbow_link: geometry visual mesh filename=meshes/right_elbow_link.STL
- link right_hand_index_0_link: geometry visual mesh filename=meshes/right_hand_index_0_link.STL
- link right_hand_index_1_link: geometry visual mesh filename=meshes/right_hand_index_1_link.STL
- link right_hand_middle_0_link: geometry visual mesh filename=meshes/right_hand_middle_0_link.STL
- link right_hand_middle_1_link: geometry visual mesh filename=meshes/right_hand_middle_1_link.STL
- link right_hand_palm_link: geometry visual mesh filename=meshes/right_hand_palm_link.STL
- link right_hand_thumb_0_link: geometry visual mesh filename=meshes/right_hand_thumb_0_link.STL
- link right_hand_thumb_1_link: geometry visual mesh filename=meshes/right_hand_thumb_1_link.STL
- link right_hand_thumb_2_link: geometry visual mesh filename=meshes/right_hand_thumb_2_link.STL
- link right_hip_pitch_link: geometry visual mesh filename=meshes/right_hip_pitch_link.STL
- link right_hip_roll_link: geometry visual mesh filename=meshes/right_hip_roll_link.STL
- link right_hip_yaw_link: geometry visual mesh filename=meshes/right_hip_yaw_link.STL
- link right_knee_link: geometry collision cylinder length=0.2 radius=0.05; visual mesh filename=meshes/right_knee_link.STL
- link right_shoulder_pitch_link: geometry visual mesh filename=meshes/right_shoulder_pitch_link.STL
- link right_shoulder_roll_link: geometry visual mesh filename=meshes/right_shoulder_roll_link.STL
- link right_shoulder_yaw_link: geometry visual mesh filename=meshes/right_shoulder_yaw_link.STL
- link right_wrist_pitch_link: geometry visual mesh filename=meshes/right_wrist_pitch_link.STL
- link right_wrist_roll_link: geometry visual mesh filename=meshes/right_wrist_roll_link.STL
- link right_wrist_yaw_link: geometry visual mesh filename=meshes/right_wrist_yaw_link.STL
